File: hardware/Filter.kicad_sch (KiCad schematic)
At the start: 0 parts

Commit message: hardware: finishing schematics
Parts:
- added C10: 100 uF 25V, symbol Device:C_Polarized
- added C3: 100 nF, symbol Device:C
- added R1, R3: R, symbol Device:R
Connections:
- new net: C10.1, C3.1, R1.2, R3.1
- new net FILTER_IN: R1.1
- new net GND: C10.2, C3.2
- new net VCC+: R3.2
