File: hardware/audio.kicad_sch (KiCad schematic)
At the start: 0 parts

Commit message: hardware: finishing schematics
Parts:
- added BATT: 6-9V, symbol Device:Battery_Cell
- added C4: 10u uF 25V, symbol Device:C_Polarized
- added C5: 10 uF 25V, symbol Device:C_Polarized
- added C6: 100 nF, symbol Device:C
- added C7: 47 nF, symbol Device:C
- added C8: 220 uF 25V, symbol Device:C_Polarized
- added C9: 100 uF 25V, symbol Device:C_Polarized
- added LS: 8R, symbol Device:Speaker
- added R4: 10R, symbol Device:R
- added SW: ON/OFF SWITCH, symbol Switch:SW_DIP_x01
- added U?: LM386, symbol Amplifier_Audio:LM386
- added VR: 30K LOG, symbol Device:R_Potentiometer
Connections:
- new net: C7.2, R4.1
- new net: C8.2, LS.1
- new net: U?.3 (+), VR.2
- new net: C7.1, C8.1, U?.5
- new net: BATT.1 (+), SW.2
- new net: C4.2, U?.1 (GAIN)
- new net: C5.1, U?.7 (BYPASS)
- new net: C4.1, U?.8 (GAIN)
- new net AUDIO_IN: VR.1
- new net GND: BATT.2 (-), C5.2, C6.2, C9.2, LS.2, R4.2, U?.2 (-), U?.4 (GND), VR.3
- new net VCC+: C6.1, C9.1, SW.1, U?.6 (V+)
Other:
- company: (none) -> UFSC
- title: (none) -> FM Receiver

Commit message: hardware: finishing layout
Parts:
- removed BATT: 6-9V, symbol Device:Battery_Cell
- removed LS: 8R, symbol Device:Speaker
- added BATT1: Conn_01x02_Female, lib:bf495, symbol Connector:Conn_01x02_Female
- added JST1: Conn_01x02_Female, Inductor_THT:L_Axial_L7.0mm_D3.3mm_P12.70mm_Horizontal_Fastron_MICC, symbol Connector:Conn_01x02_Female
- C4, C5, C8, C9: footprint (none) -> Capacitor_THT:CP_Radial_D5.0mm_P2.50mm
- C6, C7: footprint (none) -> Capacitor_THT:C_Disc_D4.3mm_W1.9mm_P5.00mm
- R4: footprint (none) -> Resistor_THT:R_Axial_DIN0207_L6.3mm_D2.5mm_P10.16mm_Horizontal
- SW1: renamed from SW; footprint (none) -> Inductor_THT:L_Axial_L7.0mm_D3.3mm_P10.16mm_Horizontal_Fastron_MICC
- U1: renamed from U?; footprint (none) -> lib:lm386
- VR1: renamed from VR; footprint (none) -> TerminalBlock:TerminalBlock_bornier-3_P5.08mm
Connections:
- net GND: now also BATT1.2 (Pin_2), JST1.2 (Pin_2)
- net at C8.2: now also JST1.1 (Pin_1)
- net at SW1.2: now also BATT1.1 (Pin_1)
Changed lines of the file:
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@@
     (stroke (width 0) (type default) (color 0 0 0 0))
   )
-  (wire (pts (xy 125.73 96.52) (xy 125.73 101.6))
+  (wire (pts (xy 125.73 93.98) (xy 125.73 101.6))
     (stroke (width 0) (type default) (color 0 0 0 0))
   )
@@
     (stroke (width 0) (type default) (color 0 0 0 0))
   )
-  (wire (pts (xy 125.73 86.36) (xy 125.73 88.9))
+  (wire (pts (xy 125.73 86.36) (xy 125.73 91.44))
     (stroke (width 0) (type default) (color 0 0 0 0))
   )
@@
     (effects (font (size 1.27 1.27)) (justify right))
   )
+  (symbol (lib_id "Connector:Conn_01x02_Female") (at 95.25 95.25 0) (unit 1)
+    (in_bom yes) (on_board yes) (fields_autoplaced)
+    (property "Reference" "JST1" (id 0) (at 96.52 95.2499 0)
+      (effects (font (size 1.27 1.27)) (justify left))
+    )
+    (property "Value" "Conn_01x02_Female" (id 1) (at 96.52 97.7899 0)
+      (effects (font (size 1.27 1.27)) (justify left))
+    )
+    (property "Footprint" "Inductor_THT:L_Axial_L7.0mm_D3.3mm_P12.70mm_Horizontal_Fastron_MICC" (id 2) (at 95.25 95.25 0)
+      (effects (font (size 1.27 1.27)) hide)
+    )
+    (property "Datasheet" "~" (id 3) (at 95.25 95.25 0)
+      (effects (font (size 1.27 1.27)) hide)
+    )
+    (pin "1")
+    (pin "2")
+  )
   (symbol (lib_id "power:GND") (at 109.22 100.33 0) (unit 1)
     (in_bom yes) (on_board yes) (fields_autoplaced)
-    (property "Reference" "#PWR?" (id 0) (at 109.22 106.68 0)
+    (property "Reference" "#PWR0108" (id 0) (at 109.22 106.68 0)
       (effects (font (size 1.27 1.27)) hide)
     )
@@
   (symbol (lib_id "power:GND") (at 90.17 100.33 0) (unit 1)
     (in_bom yes) (on_board yes) (fields_autoplaced)
-    (property "Reference" "#PWR?" (id 0) (at 90.17 106.68 0)
+    (property "Reference" "#PWR0109" (id 0) (at 90.17 106.68 0)
       (effects (font (size 1.27 1.27)) hide)
     )
@@
       (effects (font (size 1.27 1.27)) (justify left))
     )
-    (property "Footprint" "" (id 2) (at 70.612 92.71 90)
+    (property "Footprint" "Resistor_THT:R_Axial_DIN0207_L6.3mm_D2.5mm_P10.16mm_Horizontal" (id 2) (at 70.612 92.71 90)
       (effects (font (size 1.27 1.27)) hide)
     )
@@
     (pin "2")
   )
-  (symbol (lib_id "Device:Speaker") (at 95.25 95.25 0) (unit 1)
-    (in_bom yes) (on_board yes) (fields_autoplaced)
-    (property "Reference" "LS" (id 0) (at 100.33 95.2499 0)
-      (effects (font (size 1.27 1.27)) (justify left))
-    )
-    (property "Value" "8R" (id 1) (at 100.33 97.7899 0)
-      (effects (font (size 1.27 1.27)) (justify left))
-    )
-    (property "Footprint" "" (id 2) (at 95.25 100.33 0)
-      (effects (font (size 1.27 1.27)) hide)
-    )
-    (property "Datasheet" "~" (id 3) (at 94.996 96.52 0)
+  (symbol (lib_id "Connector:Conn_01x02_Female") (at 130.81 91.44 0) (unit 1)
+    (in_bom yes) (on_board yes) (fields_autoplaced)
+    (property "Reference" "BATT1" (id 0) (at 132.08 91.4399 0)
+      (effects (font (size 1.27 1.27)) (justify left))
+    )
+    (property "Value" "Conn_01x02_Female" (id 1) (at 132.08 93.9799 0)
+      (effects (font (size 1.27 1.27)) (justify left))
+    )
+    (property "Footprint" "lib:bf495" (id 2) (at 130.81 91.44 0)
+      (effects (font (size 1.27 1.27)) hide)
+    )
+    (property "Datasheet" "~" (id 3) (at 130.81 91.44 0)
       (effects (font (size 1.27 1.27)) hide)
     )
@@
   (symbol (lib_id "Device:R_Potentiometer") (at 29.21 87.63 0) (unit 1)
     (in_bom yes) (on_board yes) (fields_autoplaced)
-    (property "Reference" "VR" (id 0) (at 26.67 86.3599 0)
+    (property "Reference" "VR1" (id 0) (at 26.67 86.3599 0)
       (effects (font (size 1.27 1.27)) (justify right))
     )
@@
       (effects (font (size 1.27 1.27)) (justify right))
     )
-    (property "Footprint" "" (id 2) (at 29.21 87.63 0)
+    (property "Footprint" "TerminalBlock:TerminalBlock_bornier-3_P5.08mm" (id 2) (at 29.21 87.63 0)
       (effects (font (size 1.27 1.27)) hide)
     )
@@
       (effects (font (size 1.27 1.27)) (justify left))
     )
-    (property "Footprint" "" (id 2) (at 91.1352 87.63 0)
+    (property "Footprint" "Capacitor_THT:CP_Radial_D5.0mm_P2.50mm" (id 2) (at 91.1352 87.63 0)
       (effects (font (size 1.27 1.27)) hide)
     )
@@
   (symbol (lib_id "power:GND") (at 125.73 101.6 0) (unit 1)
     (in_bom yes) (on_board yes) (fields_autoplaced)
-    (property "Reference" "#PWR?" (id 0) (at 125.73 107.95 0)
+    (property "Reference" "#PWR0107" (id 0) (at 125.73 107.95 0)
       (effects (font (size 1.27 1.27)) hide)
     )
@@
   (symbol (lib_id "power:GND") (at 38.1 99.06 0) (unit 1)
     (in_bom yes) (on_board yes) (fields_autoplaced)
-    (property "Reference" "#PWR?" (id 0) (at 38.1 105.41 0)
+    (property "Reference" "#PWR0104" (id 0) (at 38.1 105.41 0)
       (effects (font (size 1.27 1.27)) hide)
     )
@@
     (pin "1")
   )
-  (symbol (lib_id "Device:Battery_Cell") (at 125.73 93.98 0) (unit 1)
-    (in_bom yes) (on_board yes)
-    (property "Reference" "BATT" (id 0) (at 119.38 96.52 0)
-      (effects (font (size 1.27 1.27)) (justify left))
-    )
-    (property "Value" "6-9V" (id 1) (at 119.38 99.06 0)
-      (effects (font (size 1.27 1.27)) (justify left))
-    )
-    (property "Footprint" "" (id 2) (at 125.73 92.456 90)
-      (effects (font (size 1.27 1.27)) hide)
-    )
-    (property "Datasheet" "~" (id 3) (at 125.73 92.456 90)
-      (effects (font (size 1.27 1.27)) hide)
-    )
-    (pin "1")
-    (pin "2")
-  )
   (symbol (lib_id "power:GND") (at 57.15 69.85 0) (unit 1)
     (in_bom yes) (on_board yes) (fields_autoplaced)
-    (property "Reference" "#PWR?" (id 0) (at 57.15 76.2 0)
+    (property "Reference" "#PWR0106" (id 0) (at 57.15 76.2 0)
       (effects (font (size 1.27 1.27)) hide)
     )
@@
   (symbol (lib_id "power:GND") (at 24.13 67.31 0) (unit 1)
     (in_bom yes) (on_board yes) (fields_autoplaced)
-    (property "Reference" "#PWR?" (id 0) (at 24.13 73.66 0)
+    (property "Reference" "#PWR0102" (id 0) (at 24.13 73.66 0)
       (effects (font (size 1.27 1.27)) hide)
     )
@@
       (effects (font (size 1.27 1.27)) (justify left))
     )
-    (property "Footprint" "" (id 2) (at 110.1852 86.36 0)
+    (property "Footprint" "Capacitor_THT:CP_Radial_D5.0mm_P2.50mm" (id 2) (at 110.1852 86.36 0)
       (effects (font (size 1.27 1.27)) hide)
     )
@@
   (symbol (lib_id "power:GND") (at 29.21 99.06 0) (unit 1)
     (in_bom yes) (on_board yes) (fields_autoplaced)
-    (property "Reference" "#PWR?" (id 0) (at 29.21 105.41 0)
+    (property "Reference" "#PWR0103" (id 0) (at 29.21 105.41 0)
       (effects (font (size 1.27 1.27)) hide)
     )
@@
   (symbol (lib_id "Switch:SW_DIP_x01") (at 125.73 78.74 270) (unit 1)
     (in_bom yes) (on_board yes)
-    (property "Reference" "SW" (id 0) (at 126.6329 69.1248 90))
+    (property "Reference" "SW1" (id 0) (at 126.6329 69.1248 90))
     (property "Value" "ON/OFF SWITCH" (id 1) (at 125.3629 66.5848 90))
-    (property "Footprint" "" (id 2) (at 125.73 78.74 0)
+    (property "Footprint" "Inductor_THT:L_Axial_L7.0mm_D3.3mm_P10.16mm_Horizontal_Fastron_MICC" (id 2) (at 125.73 78.74 0)
       (effects (font (size 1.27 1.27)) hide)
     )
@@
   (symbol (lib_id "power:GND") (at 46.99 99.06 0) (unit 1)
     (in_bom yes) (on_board yes) (fields_autoplaced)
-    (property "Reference" "#PWR?" (id 0) (at 46.99 105.41 0)
+    (property "Reference" "#PWR0105" (id 0) (at 46.99 105.41 0)
       (effects (font (size 1.27 1.27)) hide)
     )
@@
   (symbol (lib_id "Amplifier_Audio:LM386") (at 49.53 78.74 0) (unit 1)
     (in_bom yes) (on_board yes)
-    (property "Reference" "U?" (id 0) (at 55.88 81.28 0))
+    (property "Reference" "U1" (id 0) (at 55.88 81.28 0))
     (property "Value" "LM386" (id 1) (at 55.88 83.82 0))
-    (property "Footprint" "" (id 2) (at 52.07 76.2 0)
+    (property "Footprint" "lib:lm386" (id 2) (at 52.07 76.2 0)
       (effects (font (size 1.27 1.27)) hide)
     )
@@
     (property "Reference" "C4" (id 0) (at 57.15 93.98 90))
     (property "Value" "10u uF 25V" (id 1) (at 57.15 96.52 90))
-    (property "Footprint" "" (id 2) (at 49.53 92.4052 0)
+    (property "Footprint" "Capacitor_THT:CP_Radial_D5.0mm_P2.50mm" (id 2) (at 49.53 92.4052 0)
       (effects (font (size 1.27 1.27)) hide)
     )
@@
       (effects (font (size 1.27 1.27)) (justify left))
     )
-    (property "Footprint" "" (id 2) (at 58.1152 69.85 0)
+    (property "Footprint" "Capacitor_THT:CP_Radial_D5.0mm_P2.50mm" (id 2) (at 58.1152 69.85 0)
       (effects (font (size 1.27 1.27)) hide)
     )
@@
   (symbol (lib_id "power:GND") (at 72.39 100.33 0) (unit 1)
     (in_bom yes) (on_board yes) (fields_autoplaced)
-    (property "Reference" "#PWR?" (id 0) (at 72.39 106.68 0)
+    (property "Reference" "#PWR0110" (id 0) (at 72.39 106.68 0)
       (effects (font (size 1.27 1.27)) hide)
     )
@@
       (effects (font (size 1.27 1.27)) (justify left))
     )
-    (property "Footprint" "" (id 2) (at 25.0952 67.31 0)
+    (property "Footprint" "Capacitor_THT:C_Disc_D4.3mm_W1.9mm_P5.00mm" (id 2) (at 25.0952 67.31 0)
       (effects (font (size 1.27 1.27)) hide)
     )
@@
       (effects (font (size 1.27 1.27)) (justify left))
     )
-    (property "Footprint" "" (id 2) (at 73.3552 86.36 0)
-      (effects (font (size 1.27 1.27)) hide)
-    )
+    (property "Footprint" "Capacitor_THT:C_Disc_D4.3mm_W1.9mm_P5.00mm" (id 2) (at 73.3552 86.36 0)
+      (effects (font (size 1.27 1.27)) hide)
+    )
