File: hardware/receiver.kicad_sch (KiCad schematic)
At the start: 7 parts

Commit message: hardware: finishing schematics
Parts:
- removed C? (x4): C_Polarized, symbol Device:C_Polarized
- removed U?: BF494, TO-92_ONS, symbol bf494:BF494
- added J1: AERIAL, symbol Connector:Conn_01x01_Female
- added L1: L, symbol Device:L
- added R2: 10k, symbol Device:R
- added T1: BF494, Package_TO_SOT_THT:TO-39-3, symbol Transistor_BJT:2N2219
- added T2: BF495, TO3_BF495_NXP, symbol bf495:BF495
- added VC1: 30 pF, symbol Device:C_Variable
- C1: renamed from C?; value C -> 220 nF
- C2: renamed from C?; value C -> 2.2 nF
Connections:
- net AUDIO_IN: now reaches C2.1
- net AUDIO_IN: now also R2.2
- net GND: now reaches C2.2
- net GND: now also T1.1 (E), T2.2, VC1.2
- net FILTER_IN: now reaches C1.1
- net FILTER_IN: now also J1.1 (Pin_1), L1.1, T1.2 (B), T2.3, VC1.1
- net at C1.2: now also R2.1
- new net: L1.2, T1.3 (C), T2.1
Other:
- company: (none) -> UFSC
- title: (none) -> FM Receiver
- moved on the sheet: C1, C2

Commit message: hardware: finishing layout
Parts:
- C1, C2: footprint (none) -> Capacitor_THT:C_Disc_D4.3mm_W1.9mm_P5.00mm
- J1: footprint (none) -> MountingHole:MountingHole_2.2mm_M2_DIN965_Pad
- L1: footprint (none) -> Inductor_THT:L_Axial_L7.0mm_D3.3mm_P12.70mm_Horizontal_Fastron_MICC
- R2: footprint (none) -> Resistor_THT:R_Axial_DIN0207_L6.3mm_D2.5mm_P10.16mm_Horizontal
- T2: footprint TO3_BF495_NXP -> lib:bf495
- VC1: footprint (none) -> Capacitor_THT:CP_Radial_Tantal_D5.0mm_P5.00mm
Changed lines of the file:
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@@
       (effects (font (size 1.27 1.27)) (justify left))
     )
-    (property "Footprint" "" (id 2) (at 105.1052 60.96 0)
+    (property "Footprint" "Capacitor_THT:C_Disc_D4.3mm_W1.9mm_P5.00mm" (id 2) (at 105.1052 60.96 0)
       (effects (font (size 1.27 1.27)) hide)
     )
@@
   )
   (symbol (lib_id "Connector:Conn_01x01_Female") (at 19.05 63.5 180) (unit 1)
-    (in_bom yes) (on_board yes) (fields_autoplaced)
+    (in_bom yes) (on_board yes)
     (property "Reference" "J1" (id 0) (at 19.685 58.42 0))
     (property "Value" "AERIAL" (id 1) (at 19.685 60.96 0))
-    (property "Footprint" "" (id 2) (at 19.05 63.5 0)
+    (property "Footprint" "MountingHole:MountingHole_2.2mm_M2_DIN965_Pad" (id 2) (at 19.05 63.5 0)
       (effects (font (size 1.27 1.27)) hide)
     )
@@
     (property "Reference" "R2" (id 0) (at 96.52 36.83 90))
     (property "Value" "10k" (id 1) (at 96.52 39.37 90))
-    (property "Footprint" "" (id 2) (at 96.52 44.958 90)
+    (property "Footprint" "Resistor_THT:R_Axial_DIN0207_L6.3mm_D2.5mm_P10.16mm_Horizontal" (id 2) (at 96.52 44.958 90)
       (effects (font (size 1.27 1.27)) hide)
     )
@@
       (effects (font (size 1.27 1.27)) (justify left))
     )
-    (property "Footprint" "" (id 2) (at 27.94 69.85 0)
+    (property "Footprint" "Capacitor_THT:CP_Radial_Tantal_D5.0mm_P5.00mm" (id 2) (at 27.94 69.85 0)
       (effects (font (size 1.27 1.27)) hide)
     )
@@
       (effects (font (size 1.27 1.27)) (justify left))
     )
-    (property "Footprint" "" (id 2) (at 48.26 46.99 0)
+    (property "Footprint" "Inductor_THT:L_Axial_L7.0mm_D3.3mm_P12.70mm_Horizontal_Fastron_MICC" (id 2) (at 48.26 46.99 0)
       (effects (font (size 1.27 1.27)) hide)
     )
@@
       (effects (font (size 1.524 1.524)) (justify left))
     )
-    (property "Footprint" "TO3_BF495_NXP" (id 2) (at 63.5 53.34 0)
+    (property "Footprint" "lib:bf495" (id 2) (at 63.5 53.34 0)
       (effects (font (size 1.27 1.27) italic) hide)
     )
@@
     (property "Reference" "C1" (id 0) (at 86.36 35.56 90))
     (property "Value" "220 nF" (id 1) (at 86.36 38.1 90))
-    (property "Footprint" "" (id 2) (at 90.17 42.2148 0)
+    (property "Footprint" "Capacitor_THT:C_Disc_D4.3mm_W1.9mm_P5.00mm" (id 2) (at 90.17 42.2148 0)
       (effects (font (size 1.27 1.27)) hide)
     )
