File: hardware/fm-receiver.kicad_pcb (KiCad board)
At the start: 2 copper layers, 53.3 x 35.6 mm, 24 parts, among them J1 AERIAL, SW1 ON/OFF SWITCH, T1 BF494, T2 BF495, U1 LM386

Commit message: hardware: adding some text to facilitate
Other:
- board text added: "ANTENNA"
- board text added: "GND"
Changed lines of the file:
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@@
     (property "Sheetname" "Receiver")
     (attr exclude_from_pos_files)
-    (fp_text reference "J1" (at 0 -3.81) (layer "F.SilkS")
+    (fp_text reference "J1" (at -0.014472 -4.061594) (layer "F.SilkS")
       (effects (font (size 1 1) (thickness 0.15)))
     )
@@
   (gr_line (start 44.45 43.18) (end 44.45 78.74) (layer "Edge.Cuts") (width 0.2))
   (gr_line (start 44.45 78.74) (end 97.79 78.74) (layer "Edge.Cuts") (width 0.2))
+  (gr_text "ANTENNA" (at 46.937749 46.69621) (layer "F.SilkS")
+    (effects (font (size 0.5 0.5) (thickness 0.1)))
+  )
+  (gr_text "GND" (at 90.17 60.268104) (layer "F.SilkS")
+    (effects (font (size 0.5 0.5) (thickness 0.1)))
+  )
   (zone (net 12) (net_name "Net-(C7-Pad2)") (layer "F.Cu") (hatch edge 0.508)
     (priority 6)
